Commit message: added transmissions

File: my_legged_robots_sims/urdf/monoped_controlled.urdf (robot description, URDF)
Before this commit: robot monoped, 5 links, 4 joints
Links:
- link base: mass 0.18 -> 0.4672
- link hipassembly: mass 0.18 -> 0.1168
- link lowerleg: mass 0.18 -> 0.0292
- link lowerleg_contactsensor_link: mass 0.01 -> 0.0001
- link upperleg: mass 0.18 -> 0.1168
Joints:
- joint haa_joint: limit lower=-1.6 upper=1.6 effort=200 velocity=10.0 -> lower=-1.6 upper=1.6 effort=2000 velocity=20.0
- joint hfe_joint: limit lower=-1.6 upper=1.6 effort=200 velocity=10.0 -> lower=-1.6 upper=1.6 effort=2000 velocity=20.0
- joint kfe_joint: limit lower=-1.6 upper=1.6 effort=200 velocity=10.0 -> lower=-1.6 upper=0.0 effort=2000 velocity=20.0
